Commit message: Created Gazebo World and edited URDOF

File: description/robot.urdf.xacro (robot description, xacro)
@@ -2,3 +2,4 @@
 <robot xmlns:xacro="http://www.ros.org/wiki/xacro"  name="robot">
     <xacro:include filename="robot_core.xacro"/>
+    <xacro:include filename="gazebo_control.xacro"/>
 </robot>

File: description/robot_core.xacro (robot description, xacro)
@@ -44,4 +44,7 @@
     </xacro:inertial_box>
 </link>
+<gazebo reference="chassis">
+    <material>Gazebo/White</material>
+</gazebo>
 <!--LEFT WHEEL LINK-->
 <joint name="left_wheel_joint" type="continuous">
@@ -67,4 +70,7 @@
     </xacro:inertial_cylinder>
 </link>
+<gazebo reference="left_wheel">
+    <material>Gazebo/Blue</material>
+</gazebo>
 <!--RIGHT WHEEL LINK-->
 <joint name="right_wheel_joint" type="continuous">
@@ -90,4 +96,7 @@
     </xacro:inertial_cylinder>
 </link>
+<gazebo reference="right_wheel">
+    <material>Gazebo/Blue</material>
+</gazebo>
 <!--CASTER WHEEL LINK-->
 <joint name="caster_Wheel_joint" type="fixed">
@@ -112,3 +121,8 @@
     </xacro:inertial_sphere>
 </link>
+<gazebo reference="caster_wheel">
+    <material>Gazebo/Black</material>
+    <mu1 value="0.001"/>
+    <mu2 value="0.001"/>
+</gazebo>
 </robot>
